Commit message: add urdf endeffector support

File: applications/config/ur5e/ur.urdf.xacro (robot description, xacro)
@@ -51,3 +51,7 @@
      <origin xyz="0 0 0" rpy="0 0 3.14159265358979323846" />          <!-- position robot in the world -->
   </xacro:ur_robot>
+  <!-- <xacro:include filename="$(find applications)/urdf/end_effector.urdf.xacro"/>
+  <xacro:end-effector name="tcp" parent="$(arg tf_prefix)tool0" mesh="driller">
+     <origin xyz="0 0 0" rpy="0 0 0" />
+  </xacro:end-effector> -->
 </robot>

Commit message: refine ur.urdf.xacro

File: applications/config/ur5e/ur.urdf.xacro (robot description, xacro)
@@ -51,7 +51,7 @@
      <origin xyz="0 0 0" rpy="0 0 3.14159265358979323846" />          <!-- position robot in the world -->
   </xacro:ur_robot>
-  <!-- <xacro:include filename="$(find applications)/urdf/end_effector.urdf.xacro"/>
-  <xacro:end-effector name="tcp" parent="$(arg tf_prefix)tool0" mesh="driller">
-     <origin xyz="0 0 0" rpy="0 0 0" />
-  </xacro:end-effector> -->
+  <xacro:include filename="$(find applications)/urdf/end_effector.urdf.xacro"/>
+  <xacro:end-effector name="handpiece" parent="$(arg tf_prefix)tool0">
+     <origin xyz="0.0000505 0.0018090 0.2960264 " rpy="0.0656498 1.2033 1.5708" />
+  </xacro:end-effector>
 </robot>

File: applications/urdf/end_effector.urdf.xacro (robot description, xacro)
@@ -1,10 +1,10 @@
 <?xml version="1.0"?>
 <robot xmlns:xacro="http://wiki.ros.org/xacro">
-<xacro:macro name="end-effector" params="parent name mesh *origin">
+<xacro:macro name="end-effector" params="parent name *origin">
     <link name="${name}">
       <visual>
         <origin xyz="0 0 0" rpy="0 0 0"/>
         <geometry>
-          <mesh filename="package://applications/meshes/${mesh}.stl" scale="0.001 0.001 0.001"/>
+          <mesh filename="package://applications/meshes/${name}.stl" scale="0.001 0.001 0.001"/>
         </geometry>
       </visual>
@@ -12,5 +12,5 @@
         <origin xyz="0 0 0" rpy="0 0 0"/>
         <geometry>
-           <mesh filename="package://applications/meshes/${mesh}.stl" scale="0.001 0.001 0.001"/>
+           <mesh filename="package://applications/meshes/${name}.stl" scale="0.001 0.001 0.001"/>
         </geometry>
       </collision>
@@ -29,8 +29,14 @@
     </link>
     <joint name="${parent}-${name}" type="fixed">
-      <xacro:insert_block name="origin" />
+       <origin xyz="0 0 0" rpy="0 0 0" />
       <parent link="${parent}"/>
       <child link="${name}"/>
     </joint>
+    <link name="tcp"/>
+    <joint name="${name}-tcp" type="fixed">
+      <xacro:insert_block name="origin" />
+      <parent link="${name}"/>
+      <child link="tcp"/>
+    </joint>
 </xacro:macro>
 </robot>

Commit message: add white material in end_effector.urdf.xacro

File: applications/config/ur5e/ur.urdf.xacro (robot description, xacro)
@@ -51,7 +51,7 @@
      <origin xyz="0 0 0" rpy="0 0 3.14159265358979323846" />          <!-- position robot in the world -->
   </xacro:ur_robot>
-  <!-- <xacro:include filename="$(find applications)/urdf/end_effector.urdf.xacro"/>
+  <xacro:include filename="$(find applications)/urdf/end_effector.urdf.xacro"/>
   <xacro:end-effector name="handpiece" parent="$(arg tf_prefix)tool0">
      <origin xyz="0.0000505 0.0018090 0.2960264 " rpy="0.0656498 1.2033 1.5708" />
-  </xacro:end-effector> -->
+  </xacro:end-effector>
 </robot>

File: applications/urdf/end_effector.urdf.xacro (robot description, xacro)
@@ -1,4 +1,7 @@
 <?xml version="1.0"?>
 <robot xmlns:xacro="http://wiki.ros.org/xacro">
+  <material name="white">
+   <color rgba="1 1 1 1"/>
+  </material>
 <xacro:macro name="end-effector" params="parent name *origin">
     <link name="${name}">
@@ -8,4 +11,5 @@
           <mesh filename="package://applications/meshes/${name}.stl" scale="0.001 0.001 0.001"/>
         </geometry>
+        <material name="white"/>
       </visual>
       <collision>
